Commit message: URDF tested correct

File: URDF/SO_5DOF_ARM100_05d.SLDASM/urdf/SO_5DOF_ARM100_05d.SLDASM.urdf (robot description, URDF)
Before this commit: robot URDF_SO_5DOF_ARM100_05d.SLDASM, 7 links, 6 joints
Links:
- link Base: geometry collision mesh filename=package://SO_5DOF_ARM100_05d.SLDASM/meshes/Base.STL; visual mesh filename=package://SO_5DOF_ARM100_05d.SLDASM/meshes/Base.STL
- link Fixed_Gripper: geometry collision mesh filename=package://SO_5DOF_ARM100_05d.SLDASM/meshes/Fixed_Gripper.STL; visual mesh filename=package://SO_5DOF_ARM100_05d.SLDASM/meshes/Fixed_Gripper.STL
- link Lower_Arm: geometry collision mesh filename=package://SO_5DOF_ARM100_05d.SLDASM/meshes/Lower_Arm.STL; visual mesh filename=package://SO_5DOF_ARM100_05d.SLDASM/meshes/Lower_Arm.STL
- link Moving_Jaw: geometry collision mesh filename=package://SO_5DOF_ARM100_05d.SLDASM/meshes/Moving_Jaw.STL; visual mesh filename=package://SO_5DOF_ARM100_05d.SLDASM/meshes/Moving_Jaw.STL
- link Shoulder_Rotation_Pitch: geometry collision mesh filename=package://SO_5DOF_ARM100_05d.SLDASM/meshes/Shoulder_Rotatio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; visual mesh filename=package://SO_5DOF_ARM100_05d.SLDASM/meshes/Shoulder_Rotatio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
- link Upper_Arm: geometry collision mesh filename=package://SO_5DOF_ARM100_05d.SLDASM/meshes/Upper_Arm.STL; visual mesh filename=package://SO_5DOF_ARM100_05d.SLDASM/meshes/Upper_Arm.STL
- link Wrist_Pitch_Roll: geometry collision mesh filename=package://SO_5DOF_ARM100_05d.SLDASM/meshes/Wrist_Pitch_Roll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; visual mesh filename=package://SO_5DOF_ARM100_05d.SLDASM/meshes/Wrist_Pitch_Roll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
Joints:
- joint Elbow: axis 1 0 0 -> 0 0 1
- joint Shoulder_Pitch: axis 1 0 0 -> 0 0 1
- joint Wrist_Roll: axis 0 1 0 -> 0 0 1
