Commit message: fix SO101 URDF, add SO100 URDF, remove unnecessary SLDASM files

File: Simulation/SO101/so101.urdf (robot description, URDF)
Before this commit: robot so101, 7 links, 8 joints
Links:
- removed link moving_jaw_so101_v1
- added link jaw, mass 0.012; collision mesh filename=assets/moving_jaw_so101_v1.stl; visual mesh filename=assets/moving_jaw_so101_v1.stl
- link base: mass 1e-9 -> 0.147; geometry collision mesh filename=assets/base_motor_holder_so101_v1.stl; collision mesh filename=assets/base_so101_v2.stl
- link gripper: mass 1e-9 -> 0.087; geometry collision mesh filename=assets/sts3215_03a_v1.stl; collision mesh filename=assets/wrist_roll_follower_so101_v1.stl
- link lower_arm: geometry collision mesh filename=assets/motor_holder_so101_wrist_v1.stl; collision mesh filename=assets/sts3215_03a_v1.stl
- link shoulder: geometry collision mesh filename=assets/motor_holder_so101_base_v1.stl; collision mesh filename=assets/rotation_pitch_so101_v1.stl
- link upper_arm: geometry collision mesh filename=assets/sts3215_03a_v1.stl; collision mesh filename=assets/upper_arm_so101_v1.stl
- link wrist: geometry collision mesh filename=assets/sts3215_03a_no_horn_v1.stl; collision mesh filename=assets/wrist_roll_pitch_so101_v2.stl
Joints:
- removed joint base_frame
- removed joint gripper_frame
- joint 6: child moving_jaw_so101_v1 -> jaw
