Commit message: Add old and new simulation files for so101

File: Simulation/SO101/so101_new_calib.urdf (robot description, URDF)
Before this commit: robot so101, 7 links, 8 joints
Joints:
- joint 2: limit lower=-0.174533 upper=3.31613 effort=10 velocity=10 -> lower=-1.74533 upper=1.74533 effort=10 velocity=10; origin xyz=-0.0303992 -0.0182778 -0.0542 rpy=1.5708 8.18789e-16 3.14159 -> xyz=-0.0303992 -0.0182778 -0.0542 rpy=-1.5708 -1.5708 0
- joint 3: limit lower=-3.22886 upper=0.0872665 effort=10 velocity=10 -> lower=-1.74533 upper=1.5708 effort=10 velocity=10; origin xyz=-0.11257 -0.028 2.29417e-16 rpy=-2.26208e-15 -1.3739e-15 3.14159 -> xyz=-0.11257 -0.028 2.46331e-16 rpy=-1.22818e-15 5.75928e-16 1.5708
- joint 4: origin xyz=-0.1349 0.0052 3.21791e-16 rpy=-1.11022e-16 1.11022e-16 -1.5708 -> xyz=-0.1349 0.0052 1.65232e-16 rpy=3.2474e-15 2.86219e-15 -1.5708
- joint 5: origin xyz=-2.77556e-17 -0.0611 0.0181 rpy=1.5708 2.18394e-16 3.14159 -> xyz=0 -0.0611 0.0181 rpy=1.5708 -9.38083e-08 3.14159
- joint 6: limit lower=-0.261799 upper=1.74533 effort=10 velocity=10 -> lower=-0.174533 upper=1.74533 effort=10 velocity=10; origin xyz=0.0202 0.0188 -0.0234 rpy=1.5708 4.00612e-15 -2.2678e-16 -> xyz=0.0202 0.0188 -0.0234 rpy=1.5708 -5.14108e-17 -1.38655e-14
- joint gripper_frame: origin xyz=-0.0079 -0.000218121 -0.0981274 rpy=-1.5708 -0 -1.5708 -> xyz=-0.0079 -0.000218121 -0.0981274 rpy=-1.5708 1.97215e-31 -1.5708

Commit message: Update URDF (#83)
* fix SO101 URDF, add SO100 URDF, remove unnecessary SLDASM files

* update SO100 URDF

* update README

File: Simulation/SO101/so101_new_calib.urdf (robot description, URDF)
Before this commit: robot so101_new_calib, 7 links, 8 joints
Links:
- removed link moving_jaw_so101_v1
- added link jaw, mass 0.012; collision mesh filename=assets/moving_jaw_so101_v1.stl; visual mesh filename=assets/moving_jaw_so101_v1.stl
- link base: mass 1e-9 -> 0.147; geometry collision mesh filename=assets/base_motor_holder_so101_v1.stl; collision mesh filename=assets/base_so101_v2.stl
- link gripper: mass 1e-9 -> 0.087; geometry collision mesh filename=assets/sts3215_03a_v1.stl; collision mesh filename=assets/wrist_roll_follower_so101_v1.stl
- link lower_arm: geometry collision mesh filename=assets/motor_holder_so101_wrist_v1.stl; collision mesh filename=assets/sts3215_03a_v1.stl
- link shoulder: geometry collision mesh filename=assets/motor_holder_so101_base_v1.stl; collision mesh filename=assets/rotation_pitch_so101_v1.stl
- link upper_arm: geometry collision mesh filename=assets/sts3215_03a_v1.stl; collision mesh filename=assets/upper_arm_so101_v1.stl
- link wrist: geometry collision mesh filename=assets/sts3215_03a_no_horn_v1.stl; collision mesh filename=assets/wrist_roll_pitch_so101_v2.stl
Joints:
- removed joint base_frame
- removed joint gripper_frame
- joint 6: child moving_jaw_so101_v1 -> jaw

File: Simulation/SO101/so101_old_calib.urdf (robot description, URDF)
Before this commit: robot so101_old_calib, 7 links, 8 joints
Links:
- removed link moving_jaw_so101_v1
- added link jaw, mass 0.012; collision mesh filename=assets/moving_jaw_so101_v1.stl; visual mesh filename=assets/moving_jaw_so101_v1.stl
- link base: mass 1e-9 -> 0.147; geometry collision mesh filename=assets/base_motor_holder_so101_v1.stl; collision mesh filename=assets/base_so101_v2.stl
- link gripper: mass 1e-9 -> 0.087; geometry collision mesh filename=assets/sts3215_03a_v1.stl; collision mesh filename=assets/wrist_roll_follower_so101_v1.stl
- link lower_arm: geometry collision mesh filename=assets/motor_holder_so101_wrist_v1.stl; collision mesh filename=assets/sts3215_03a_v1.stl
- link shoulder: geometry collision mesh filename=assets/motor_holder_so101_base_v1.stl; collision mesh filename=assets/rotation_pitch_so101_v1.stl
- link upper_arm: geometry collision mesh filename=assets/sts3215_03a_v1.stl; collision mesh filename=assets/upper_arm_so101_v1.stl
- link wrist: geometry collision mesh filename=assets/sts3215_03a_no_horn_v1.stl; collision mesh filename=assets/wrist_roll_pitch_so101_v2.stl
Joints:
- removed joint base_frame
- removed joint gripper_frame
- joint 6: child moving_jaw_so101_v1 -> jaw

Commit message: (update) updated the new so101 calibration urdf with fixed direction and frame names

File: Simulation/SO101/so101_new_calib.urdf (robot description, URDF)
Before this commit: robot so101_new_calib, 7 links, 6 joints
Links:
- removed link jaw
- added link baseframe, mass 1e-9
- added link gripperframe, mass 1e-9
- added link moving_jaw_so101_v1, mass 0.012; collision mesh filename=package://assets/moving_jaw_so101_v1.stl; visual mesh filename=package://assets/moving_jaw_so101_v1.stl
- link base: geometry collision mesh filename=package://assets/base_motor_holder_so101_v1.stl; collision mesh filename=package://assets/base_so101_v2.stl
- link gripper: geometry collision mesh filename=package://assets/sts3215_03a_v1.stl; collision mesh filename=package://assets/wrist_roll_follower_so101_v1.stl
- link lower_arm: geometry collision mesh filename=package://assets/motor_holder_so101_wrist_v1.stl; collision mesh filename=package://assets/sts3215_03a_v1.stl
- link shoulder: geometry collision mesh filename=package://assets/motor_holder_so101_base_v1.stl; collision mesh filename=package://assets/rotation_pitch_so101_v1.stl
- link upper_arm: geometry collision mesh filename=package://assets/sts3215_03a_v1.stl; collision mesh filename=package://assets/upper_arm_so101_v1.stl
- link wrist: geometry collision mesh filename=package://assets/sts3215_03a_no_horn_v1.stl; collision mesh filename=package://assets/wrist_roll_pitch_so101_v2.stl
Joints:
- added joint baseframe_frame: type fixed, parent base, child baseframe, origin xyz=-0.163038 -0.168068 0.0324817 rpy=1.6144e-15 7.84513e-18 1.33799e-15, axis 0 0 0
- added joint gripperframe_frame: type fixed, parent gripper, child gripperframe, origin xyz=-0.0079 -0.000218121 -0.0981274 rpy=-0 1.5708 0, axis 0 0 0
- joint 1: origin xyz=0.0207909 -0.0230745 0.0948817 rpy=-3.14159 6.03684e-16 1.5708 -> xyz=-0.124202 -0.168068 0.0948817 rpy=3.14159 4.18253e-17 -3.14159
- joint 3: origin xyz=-0.11257 -0.028 2.46331e-16 rpy=-1.22818e-15 5.75928e-16 1.5708 -> xyz=-0.11257 -0.028 2.09886e-16 rpy=-3.63608e-16 8.74301e-16 1.5708
- joint 4: origin xyz=-0.1349 0.0052 1.65232e-16 rpy=3.2474e-15 2.86219e-15 -1.5708 -> xyz=-0.1349 0.0052 8.44651e-17 rpy=4.02456e-15 8.67362e-16 -1.5708
- joint 5: limit lower=-2.79253 upper=2.79253 effort=10 velocity=10 -> lower=-2.74385 upper=2.84121 effort=10 velocity=10; origin xyz=0 -0.0611 0.0181 rpy=1.5708 -9.38083e-08 3.14159 -> xyz=2.77556e-16 -0.0611 0.0181 rpy=1.5708 0.0486795 3.14159
- joint 6: child jaw -> moving_jaw_so101_v1; origin xyz=0.0202 0.0188 -0.0234 rpy=1.5708 -5.14108e-17 -1.38655e-14 -> xyz=0.0202 0.0188 -0.0234 rpy=1.5708 -5.24284e-08 -1.41553e-15

Commit message: Re-integrate the latest changes in the urdf"  1- remove package in assets path  2- add material back  3- add encoding style in xml header

File: Simulation/SO101/so101_new_calib.urdf (robot description, URDF)
Before this commit: robot so101_new_calib, 9 links, 8 joints
Links:
- link base: geometry collision mesh filename=assets/base_motor_holder_so101_v1.stl; collision mesh filename=assets/base_so101_v2.stl
- link gripper: geometry collision mesh filename=assets/sts3215_03a_v1.stl; collision mesh filename=assets/wrist_roll_follower_so101_v1.stl
- link lower_arm: geometry collision mesh filename=assets/motor_holder_so101_wrist_v1.stl; collision mesh filename=assets/sts3215_03a_v1.stl
- link moving_jaw_so101_v1: geometry collision mesh filename=assets/moving_jaw_so101_v1.stl; visual mesh filename=assets/moving_jaw_so101_v1.stl
- link shoulder: geometry collision mesh filename=assets/motor_holder_so101_base_v1.stl; collision mesh filename=assets/rotation_pitch_so101_v1.stl
- link upper_arm: geometry collision mesh filename=assets/sts3215_03a_v1.stl; collision mesh filename=assets/upper_arm_so101_v1.stl
- link wrist: geometry collision mesh filename=assets/sts3215_03a_no_horn_v1.stl; collision mesh filename=assets/wrist_roll_pitch_so101_v2.stl

Commit message: Place back the pose of the so101_new_calib to adhere to the same conventions used in the other description files

File: Simulation/SO101/so101_new_calib.urdf (robot description, URDF)
Before this commit: robot so101_new_calib, 9 links, 8 joints
Joints:
- joint 1: origin xyz=-0.124202 -0.168068 0.0948817 rpy=3.14159 4.18253e-17 -3.14159 -> xyz=0.0207909 -0.0230745 0.0948817 rpy=-3.14159 6.03684e-16 1.5708
- joint 3: origin xyz=-0.11257 -0.028 2.09886e-16 rpy=-3.63608e-16 8.74301e-16 1.5708 -> xyz=-0.11257 -0.028 2.46331e-16 rpy=-1.22818e-15 5.75928e-16 1.5708
- joint 4: origin xyz=-0.1349 0.0052 8.44651e-17 rpy=4.02456e-15 8.67362e-16 -1.5708 -> xyz=-0.1349 0.0052 1.65232e-16 rpy=3.2474e-15 2.86219e-15 -1.5708
- joint 5: limit lower=-2.74385 upper=2.84121 effort=10 velocity=10 -> lower=-2.79253 upper=2.79253 effort=10 velocity=10; origin xyz=2.77556e-16 -0.0611 0.0181 rpy=1.5708 0.0486795 3.14159 -> xyz=0 -0.0611 0.0181 rpy=1.5708 -9.38083e-08 3.14159
- joint 6: origin xyz=0.0202 0.0188 -0.0234 rpy=1.5708 -5.24284e-08 -1.41553e-15 -> xyz=0.0202 0.0188 -0.0234 rpy=1.5708 -5.14108e-17 -1.38655e-14
- joint baseframe_frame: origin xyz=-0.163038 -0.168068 0.0324817 rpy=1.6144e-15 7.84513e-18 1.33799e-15 -> xyz=0.020791 0.0157608 0.0324817 rpy=2.77556e-17 -9.52796e-30 -2.64454e-46
- joint gripperframe_frame: origin xyz=-0.0079 -0.000218121 -0.0981274 rpy=-0 1.5708 0 -> xyz=-0.0079 -0.000218121 -0.0981274 rpy=1.5708 1.22465e-16 1.5708

Commit message: shift joint(3) elbow flex by five degrees to adhere to the offset on the real robot

File: Simulation/SO101/so101_new_calib.urdf (robot description, URDF)
Before this commit: robot so101_new_calib, 9 links, 8 joints
Joints:
- joint 3: limit lower=-1.74533 upper=1.5708 effort=10 velocity=10 -> lower=-1.6580 upper=1.6581 effort=10 velocity=10

Commit message: correct joint 3 offset

File: Simulation/SO101/so101_new_calib.urdf (robot description, URDF)
Before this commit: robot so101_new_calib, 9 links, 8 joints
Joints:
- joint 3: limit lower=-1.6580 upper=1.6581 effort=10 velocity=10 -> lower=-1.69 upper=1.69 effort=10 velocity=10

Commit message: fix(joints ranges): Fixing ctrlrange to match joints limits, unifying joints limitis between URDF and XML files

File: Simulation/SO101/so101_new_calib.urdf (robot description, URDF)
Before this commit: robot so101_new_calib, 9 links, 8 joints
Joints:
- joint wrist_roll: limit lower=-2.79253 upper=2.79253 effort=10 velocity=10 -> lower=-2.74385 upper=2.84121 effort=10 velocity=10

Commit message: Updated the new so101 calibration urdf with fixed direction and frame (#106)
* (update) updated the new so101 calibration urdf with fixed direction and frame names

* Re-integrate the latest changes in the urdf"
 1- remove package in assets path
 2- add material back
 3- add encoding style in xml header

* Add back blocks related to transmissions

* Place back the pose of the so101_new_calib to adhere to the same conventions used in the other description files

* add ctrlrange to the xml file to control each joint of so101_new_calib over the full range of motion

* shift joint(3) elbow flex by five degrees to adhere to the offset on the real robot

* correct joint 3 offset

* style(joints names): Renamming joints to match LeRobot middleware naming convention

* fix(joints ranges): Fixing ctrlrange to match joints limits, unifying joints limitis between URDF and XML files

* fix(joints ranges): Fixing ctrlrange to match joints limits, unifying joints limitis between URDF and XML files

---------

Co-authored-by: CarolinePascal <caroline8.pascal@gmail.com>

File: Simulation/SO101/so101_new_calib.urdf (robot description, URDF)
Before this commit: robot so101_new_calib, 7 links, 6 joints
Links:
- removed link jaw
- added link baseframe, mass 1e-9
- added link gripperframe, mass 1e-9
- added link moving_jaw_so101_v1, mass 0.012; collision mesh filename=assets/moving_jaw_so101_v1.stl; visual mesh filename=assets/moving_jaw_so101_v1.stl
Joints:
- removed joint 1
- removed joint 2
- removed joint 3
- removed joint 4
- removed joint 5
- removed joint 6
- added joint baseframe_frame: type fixed, parent base, child baseframe, origin xyz=0.020791 0.0157608 0.0324817 rpy=2.77556e-17 -9.52796e-30 -2.64454e-46, axis 0 0 0
- added joint elbow_flex: type revolute, parent upper_arm, child lower_arm, origin xyz=-0.11257 -0.028 2.46331e-16 rpy=-1.22818e-15 5.75928e-16 1.5708, axis 0 0 1, limit lower=-1.69 upper=1.69 effort=10 velocity=10
- added joint gripper: type revolute, parent gripper, child moving_jaw_so101_v1, origin xyz=0.0202 0.0188 -0.0234 rpy=1.5708 -5.14108e-17 -1.38655e-14, axis 0 0 1, limit lower=-0.174533 upper=1.74533 effort=10 velocity=10
- added joint gripperframe_frame: type fixed, parent gripper, child gripperframe, origin xyz=-0.0079 -0.000218121 -0.0981274 rpy=1.5708 1.22465e-16 1.5708, axis 0 0 0
- added joint shoulder_lift: type revolute, parent shoulder, child upper_arm, origin xyz=-0.0303992 -0.0182778 -0.0542 rpy=-1.5708 -1.5708 0, axis 0 0 1, limit lower=-1.74533 upper=1.74533 effort=10 velocity=10
- added joint shoulder_pan: type revolute, parent base, child shoulder, origin xyz=0.0207909 -0.0230745 0.0948817 rpy=-3.14159 6.03684e-16 1.5708, axis 0 0 1, limit lower=-1.91986 upper=1.91986 effort=10 velocity=10
- added joint wrist_flex: type revolute, parent lower_arm, child wrist, origin xyz=-0.1349 0.0052 1.65232e-16 rpy=3.2474e-15 2.86219e-15 -1.5708, axis 0 0 1, limit lower=-1.65806 upper=1.65806 effort=10 velocity=10
- added joint wrist_roll: type revolute, parent wrist, child gripper, origin xyz=0 -0.0611 0.0181 rpy=1.5708 -9.38083e-08 3.14159, axis 0 0 1, limit lower=-2.74385 upper=2.84121 effort=10 velocity=10

Commit message: fix(urdf): fixing multiple issues related to the last URDF update
* Adding _link suffix to link names to avoid duplicates

* Removing unused intermediate base frame

* Fixing origin frame offsets

File: Simulation/SO101/so101_new_calib.urdf (robot description, URDF)
Before this commit: robot so101_new_calib, 9 links, 8 joints
Links:
- removed link base
- removed link baseframe
- removed link gripper
- removed link gripperframe
- removed link lower_arm
- removed link moving_jaw_so101_v1
- removed link shoulder
- removed link upper_arm
- removed link wrist
- added link base_link, mass 0.147; collision mesh filename=assets/base_motor_holder_so101_v1.stl; collision mesh filename=assets/base_so101_v2.stl
- added link gripper_frame_link, mass 1e-9
- added link gripper_link, mass 0.087; collision mesh filename=assets/sts3215_03a_v1.stl; collision mesh filename=assets/wrist_roll_follower_so101_v1.stl
- added link lower_arm_link, mass 0.104; collision mesh filename=assets/motor_holder_so101_wrist_v1.stl; collision mesh filename=assets/sts3215_03a_v1.stl
- added link moving_jaw_so101_v1_link, mass 0.012; collision mesh filename=assets/moving_jaw_so101_v1.stl; visual mesh filename=assets/moving_jaw_so101_v1.stl
- added link shoulder_link, mass 0.100006; collision mesh filename=assets/motor_holder_so101_base_v1.stl; collision mesh filename=assets/rotation_pitch_so101_v1.stl
- added link upper_arm_link, mass 0.103; collision mesh filename=assets/sts3215_03a_v1.stl; collision mesh filename=assets/upper_arm_so101_v1.stl
- added link wrist_link, mass 0.079; collision mesh filename=assets/sts3215_03a_no_horn_v1.stl; collision mesh filename=assets/wrist_roll_pitch_so101_v2.stl
Joints:
- removed joint baseframe_frame
- removed joint gripperframe_frame
- added joint gripper_frame_joint: type fixed, parent gripper_link, child gripper_frame_link, origin xyz=-0.0079 -0.000218121 -0.0981274 rpy=0 3.14159 0, axis 0 0 0
- joint elbow_flex: child lower_arm -> lower_arm_link; origin xyz=-0.11257 -0.028 2.46331e-16 rpy=-1.22818e-15 5.75928e-16 1.5708 -> xyz=-0.11257 -0.028 1.73763e-16 rpy=-3.63608e-16 8.74301e-16 1.5708; parent upper_arm -> upper_arm_link
- joint gripper: child moving_jaw_so101_v1 -> moving_jaw_so101_v1_link; origin xyz=0.0202 0.0188 -0.0234 rpy=1.5708 -5.14108e-17 -1.38655e-14 -> xyz=0.0202 0.0188 -0.0234 rpy=1.5708 -5.24284e-08 -1.41553e-15; parent gripper -> gripper_link
- joint shoulder_lift: child upper_arm -> upper_arm_link; parent shoulder -> shoulder_link
- joint shoulder_pan: child shoulder -> shoulder_link; origin xyz=0.0207909 -0.0230745 0.0948817 rpy=-3.14159 6.03684e-16 1.5708 -> xyz=0.0388353 -8.97657e-09 0.0624 rpy=3.14159 4.18253e-17 -3.14159; parent base -> base_link
- joint wrist_flex: child wrist -> wrist_link; origin xyz=-0.1349 0.0052 1.65232e-16 rpy=3.2474e-15 2.86219e-15 -1.5708 -> xyz=-0.1349 0.0052 3.62355e-17 rpy=4.02456e-15 8.67362e-16 -1.5708; parent lower_arm -> lower_arm_link
- joint wrist_roll: child gripper -> gripper_link; origin xyz=0 -0.0611 0.0181 rpy=1.5708 -9.38083e-08 3.14159 -> xyz=5.55112e-17 -0.0611 0.0181 rpy=1.5708 0.0486795 3.14159; parent wrist -> wrist_link

Commit message: better joint limits

File: Simulation/SO101/so101_new_calib.urdf (robot description, URDF)
Before this commit: robot so101_new_calib, 8 links, 7 joints
Joints:
- joint elbow_flex: limit lower=-1.69 upper=1.69 effort=10 velocity=10 -> lower=-1.81448 upper=1.57339 effort=10 velocity=10
- joint gripper: limit lower=-0.174533 upper=1.74533 effort=10 velocity=10 -> lower=-0.19990 upper=2.00767 effort=10 velocity=10
- joint shoulder_lift: limit lower=-1.74533 upper=1.74533 effort=10 velocity=10 -> lower=-1.82697 upper=1.76783 effort=10 velocity=10
- joint shoulder_pan: limit lower=-1.91986 upper=1.91986 effort=10 velocity=10 -> lower=-2.01012 upper=2.15186 effort=10 velocity=10
- joint wrist_flex: limit lower=-1.65806 upper=1.65806 effort=10 velocity=10 -> lower=-1.81662 upper=1.77853 effort=10 velocity=10
- joint wrist_roll: limit lower=-2.74385 upper=2.84121 effort=10 velocity=10 -> lower=-3.14159 upper=3.14159 effort=10 velocity=10
