Commit message: update SO100 URDF

File: Simulation/SO100/so100.urdf (robot description, URDF)
Before this commit: robot so_arm100, 7 links, 6 joints
Joints:
- removed joint Elbow
- removed joint Pitch
- removed joint Rotation
- removed joint Wrist_Pitch
- added joint 1: type revolute, parent base, child shoulder, origin xyz=0 -0.0452 0.0165 rpy=1.57079 0 0, axis 0 1 0, limit lower=-2 upper=2 effort=35 velocity=1
- added joint 2: type revolute, parent shoulder, child upper_arm, origin xyz=0 0.1025 0.0306 rpy=-1.8 0 0, axis 1 0 0, limit lower=0 upper=3.5 effort=35 velocity=1
- added joint 3: type revolute, parent upper_arm, child lower_arm, origin xyz=0 0.11257 0.028 rpy=1.57079 0 0, axis 1 0 0, limit lower=-3.14158 upper=0 effort=35 velocity=1
- added joint 4: type revolute, parent lower_arm, child wrist, origin xyz=0 0.0052 0.1349 rpy=-1 0 0, axis 1 0 0, limit lower=-2.5 upper=1.2 effort=35 velocity=1

Commit message: match new lerobot angles

File: Simulation/SO100/so100.urdf (robot description, URDF)
Before this commit: robot so_arm100, 7 links, 6 joints
Joints:
- joint 1: axis 0 1 0 -> 0 -1 0
- joint 2: limit lower=0 upper=3.5 effort=35 velocity=1 -> lower=-1.75 upper=1.75 effort=35 velocity=1; origin xyz=0 0.1025 0.0306 rpy=-1.8 0 0 -> xyz=0 0.1025 0.0306 rpy=-0.05 0 0
- joint 3: limit lower=-3.14158 upper=0 effort=35 velocity=1 -> lower=-1.57079 upper=1.57079 effort=35 velocity=1; origin xyz=0 0.11257 0.028 rpy=1.57079 0 0 -> xyz=0 0.11257 0.028 rpy=0 0 0
- joint 4: limit lower=-2.5 upper=1.2 effort=35 velocity=1 -> lower=-1.9764 upper=1.7236 effort=35 velocity=1; origin xyz=0 0.0052 0.1349 rpy=-1 0 0 -> xyz=0 0.0052 0.1349 rpy=-1.5236 0 0
- joint 6: limit lower=-0.2 upper=2.0 effort=35 velocity=1 -> lower=-1.1 upper=1.1 effort=35 velocity=1; origin xyz=-0.0202 -0.0244 0 rpy=0 3.14158 0 -> xyz=-0.0202 -0.0244 0 rpy=0 3.14158 -0.9

Commit message: correct wrist and gripper joints

File: Simulation/SO100/so100.urdf (robot description, URDF)
Before this commit: robot so_arm100, 7 links, 6 joints
Joints:
- joint 5: origin xyz=0 -0.0601 0 rpy=0 1.57079 0 -> xyz=0 -0.0601 0 rpy=0 3.14158 0
- joint 6: limit lower=-1.1 upper=1.1 effort=35 velocity=1 -> lower=-0.2 upper=2.0 effort=35 velocity=1; origin xyz=-0.0202 -0.0244 0 rpy=0 3.14158 -0.9 -> xyz=-0.0202 -0.0244 0 rpy=0 3.14158 0

Commit message: style(joints names): Renamming joints to match LeRobot middleware naming convention

File: Simulation/SO100/so100.urdf (robot description, URDF)
Before this commit: robot so_arm100, 7 links, 6 joints
Joints:
- removed joint 1
- removed joint 2
- removed joint 3
- removed joint 4
- removed joint 5
- removed joint 6
- added joint elbow_flex: type revolute, parent upper_arm, child lower_arm, origin xyz=0 0.11257 0.028 rpy=1.57079 0 0, axis 1 0 0, limit lower=-3.14158 upper=0 effort=35 velocity=1
- added joint gripper: type revolute, parent gripper, child jaw, origin xyz=-0.0202 -0.0244 0 rpy=0 3.14158 0, axis 0 0 1, limit lower=-0.2 upper=2.0 effort=35 velocity=1
- added joint shoulder_lift: type revolute, parent shoulder, child upper_arm, origin xyz=0 0.1025 0.0306 rpy=-1.8 0 0, axis 1 0 0, limit lower=0 upper=3.5 effort=35 velocity=1
- added joint shoulder_pan: type revolute, parent base, child shoulder, origin xyz=0 -0.0452 0.0165 rpy=1.57079 0 0, axis 0 1 0, limit lower=-2 upper=2 effort=35 velocity=1
- added joint wrist_flex: type revolute, parent lower_arm, child wrist, origin xyz=0 0.0052 0.1349 rpy=-1 0 0, axis 1 0 0, limit lower=-2.5 upper=1.2 effort=35 velocity=1
- added joint wrist_roll: type revolute, parent wrist, child gripper, origin xyz=0 -0.0601 0 rpy=0 1.57079 0, axis 0 1 0, limit lower=-3.14158 upper=3.14158 effort=35 velocity=1

File: Simulation/SO101/so101_new_calib.urdf (robot description, URDF)
Before this commit: robot so101_new_calib, 9 links, 8 joints
Joints:
- removed joint 1
- removed joint 2
- removed joint 3
- removed joint 4
- removed joint 5
- removed joint 6
- added joint elbow_flex: type revolute, parent upper_arm, child lower_arm, origin xyz=-0.11257 -0.028 2.46331e-16 rpy=-1.22818e-15 5.75928e-16 1.5708, axis 0 0 1, limit lower=-1.69 upper=1.69 effort=10 velocity=10
- added joint gripper: type revolute, parent gripper, child moving_jaw_so101_v1, origin xyz=0.0202 0.0188 -0.0234 rpy=1.5708 -5.14108e-17 -1.38655e-14, axis 0 0 1, limit lower=-0.174533 upper=1.74533 effort=10 velocity=10
- added joint shoulder_lift: type revolute, parent shoulder, child upper_arm, origin xyz=-0.0303992 -0.0182778 -0.0542 rpy=-1.5708 -1.5708 0, axis 0 0 1, limit lower=-1.74533 upper=1.74533 effort=10 velocity=10
- added joint shoulder_pan: type revolute, parent base, child shoulder, origin xyz=0.0207909 -0.0230745 0.0948817 rpy=-3.14159 6.03684e-16 1.5708, axis 0 0 1, limit lower=-1.91986 upper=1.91986 effort=10 velocity=10
- added joint wrist_flex: type revolute, parent lower_arm, child wrist, origin xyz=-0.1349 0.0052 1.65232e-16 rpy=3.2474e-15 2.86219e-15 -1.5708, axis 0 0 1, limit lower=-1.65806 upper=1.65806 effort=10 velocity=10
- added joint wrist_roll: type revolute, parent wrist, child gripper, origin xyz=0 -0.0611 0.0181 rpy=1.5708 -9.38083e-08 3.14159, axis 0 0 1, limit lower=-2.79253 upper=2.79253 effort=10 velocity=10

File: Simulation/SO101/so101_old_calib.urdf (robot description, URDF)
Before this commit: robot so101_old_calib, 7 links, 6 joints
Joints:
- removed joint 1
- removed joint 2
- removed joint 3
- removed joint 4
- removed joint 5
- removed joint 6
- added joint elbow_flex: type revolute, parent upper_arm, child lower_arm, origin xyz=-0.028 0.11257 1.24466e-16 rpy=1.89432e-15 -3.22659e-15 -3.14159, axis 0 0 1, limit lower=-0.174533 upper=3.14159 effort=10 velocity=10
- added joint gripper: type revolute, parent gripper, child jaw, origin xyz=0.0202 0.0188 -0.0234 rpy=1.5708 -7.91661e-17 -1.0396e-16, axis 0 0 1, limit lower=-0.174533 upper=1.74533 effort=10 velocity=10
- added joint shoulder_lift: type revolute, parent shoulder, child upper_arm, origin xyz=-0.0303992 -0.0182778 -0.0542 rpy=-1.5708 1.5708 0, axis 0 0 1, limit lower=-3.31613 upper=0.174533 effort=10 velocity=10
- added joint shoulder_pan: type revolute, parent base, child shoulder, origin xyz=0.0207909 -0.0230745 0.0948817 rpy=-3.14159 6.03684e-16 1.5708, axis 0 0 1, limit lower=-1.91986 upper=1.91986 effort=10 velocity=10
- added joint wrist_flex: type revolute, parent lower_arm, child wrist, origin xyz=-0.0052 -0.1349 3.40439e-16 rpy=-1.41553e-15 4.91611e-15 7.56157e-09, axis 0 0 1, limit lower=-1.65806 upper=1.65806 effort=10 velocity=10
- added joint wrist_roll: type revolute, parent wrist, child gripper, origin xyz=2.77556e-17 -0.0611 0.0181 rpy=1.5708 -9.38083e-08 3.14159, axis 0 0 1, limit lower=-2.79253 upper=2.79253 effort=10 velocity=10
